File: KICAD/packer.kicad_sch (KiCad schematic)
At the start: 18 parts, among them SW1 押出, SW2 戻, SW3 ゲート開, SW4 ゲート閉, SW5 排出シーケンス, SW6 反転, SW7 下降, SW8 掻込, SW9 上昇

Commit message: img
Connections:
- net 閉 　近接: now also arduino_nano1. (VIN)
- new net: 4CH_RELAY1. (IN4), arduino_nano1. (VIN) (x4)
- new net: 6CH_RELAY. (NC6), arduino_nano1. (VIN) (x6)
